File: hardware/adapter.kicad_pcb (KiCad board)
At the start: 2 copper layers, 63 parts

Commit message: Minorchanges on hardware plate
Routing:
- net (no net): track 2091.5 -> 2095.2 mm, vias 34 -> 33
Changed lines of the file:
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@@
   (general
     (thickness 1.6)
-    (drawings 4)
-    (tracks 466)
+    (drawings 7)
+    (tracks 464)
     (zones 0)
     (modules 63)
@@
     )
   )
+  (gr_poly (pts (xy 64.77 17.78) (xy 62.23 20.32) (xy 62.23 15.24) (xy 64.77 15.24)) (layer Cmts.User) (width 0.1))
+  (gr_poly (pts (xy 74.93 57.15) (xy 72.39 57.15) (xy 72.39 50.8) (xy 74.93 48.26)) (layer Cmts.User) (width 0.1))
+  (gr_poly (pts (xy 92.71 78.74) (xy 88.9 78.74) (xy 88.9 73.66) (xy 92.71 73.66)) (layer Cmts.User) (width 0.1))
   (gr_poly (pts (xy 87.63 26.67) (xy 85.09 26.67) (xy 83.82 15.24) (xy 87.63 15.24)) (layer Cmts.User) (width 0.1))
   (gr_poly (pts (xy 148.59 33.02) (xy 140.97 33.02) (xy 140.97 27.94) (xy 148.59 27.94)) (layer Cmts.User) (width 0.1))
@@
   (segment (start 82.55 68.58) (end 87.63 68.58) (width 1.4) (layer F.Cu) (net 0))
   (segment (start 91.44 71.12) (end 85.09 71.12) (width 1.4) (layer F.Cu) (net 0))
-  (segment (start 85.09 74.93) (end 85.09 71.12) (width 1.4) (layer F.Cu) (net 0))
-  (segment (start 86.36 76.2) (end 85.09 74.93) (width 1.4) (layer F.Cu) (net 0))
   (via (at 88.9 73.66) (size 2) (drill 1) (layers F.Cu B.Cu) (net 0))
   (via (at 88.9 59.69) (size 2) (drill 1) (layers F.Cu B.Cu) (net 0))
   (segment (start 88.9 73.66) (end 91.44 73.66) (width 1.4) (layer F.Cu) (net 0))
   (segment (start 91.44 57.15) (end 88.9 59.69) (width 1.4) (layer F.Cu) (net 0))
-  (via (at 88.9 78.74) (size 2) (drill 1) (layers F.Cu B.Cu) (net 0))
   (segment (start 78.74 63.5) (end 85.09 63.5) (width 1.4) (layer F.Cu) (net 0))
   (segment (start 59.69 67.31) (end 59.69 57.15) (width 1.4) (layer F.Cu) (net 0))
@@
   (segment (start 99.06 68.58) (end 107.95 68.58) (width 1.4) (layer F.Cu) (net 0))
   (segment (start 88.9 59.69) (end 88.9 73.66) (width 1.4) (layer B.Cu) (net 0))
-  (segment (start 88.9 73.66) (end 88.9 78.74) (width 1.4) (layer B.Cu) (net 0))
-  (segment (start 123.19 76.2) (end 125.73 76.2) (width 1.4) (layer F.Cu) (net 0))
   (segment (start 133.35 76.2) (end 139.7 76.2) (width 1.4) (layer F.Cu) (net 0))
   (segment (start 139.7 76.2) (end 139.7 72.39) (width 1.4) (layer F.Cu) (net 0))
@@
   (segment (start 142.24 76.2) (end 146.05 76.2) (width 1.4) (layer F.Cu) (net 0))
   (segment (start 88.9 78.74) (end 101.6 78.74) (width 1.4) (layer F.Cu) (net 0))
-  (segment (start 122.555 75.565) (end 121.92 74.93) (width 1.4) (layer F.Cu) (net 0))
-  (segment (start 123.19 76.2) (end 122.555 75.565) (width 1.4) (layer F.Cu) (net 0))
   (segment (start 137.16 64.77) (end 133.35 64.77) (width 1.4) (layer F.Cu) (net 0))
   (segment (start 133.35 64.77) (end 130.81 62.23) (width 1.4) (layer F.Cu) (net 0))
@@
   (segment (start 118.11 19.05) (end 119.38 20.32) (width 1.4) (layer F.Cu) (net 0))
   (segment (start 114.3 52.07) (end 116.84 52.07) (width 1.4) (layer F.Cu) (net 0))
-  (segment (start 121.92 74.93) (end 116.84 74.93) (width 1.4) (layer F.Cu) (net 0))
   (segment (start 110.49 68.58) (end 110.49 69.85) (width 1.4) (layer F.Cu) (net 0))
   (segment (start 104.14 68.58) (end 110.49 68.58) (width 1.4) (layer F.Cu) (net 0))
@@
   (segment (start 97.79 62.23) (end 99.06 63.5) (width 1.4) (layer F.Cu) (net 0))
   (segment (start 113.03 73.66) (end 114.3 72.39) (width 1.4) (layer F.Cu) (net 0))
-  (segment (start 86.36 76.2) (end 106.68 76.2) (width 1.4) (layer F.Cu) (net 0))
-  (segment (start 102.87 76.2) (end 115.57 76.2) (width 1.4) (layer F.Cu) (net 0))
   (segment (start 115.57 76.2) (end 116.84 74.93) (width 1.4) (layer F.Cu) (net 0))
   (segment (start 119.38 71.12) (end 120.65 72.39) (width 1.4) (layer F.Cu) (net 0))
@@
   (segment (start 110.49 66.04) (end 111.76 64.77) (width 1.4) (layer F.Cu) (net 0))
   (segment (start 110.49 68.58) (end 110.49 66.04) (width 1.4) (layer F.Cu) (net 0))
-  (segment (start 123.19 74.93) (end 122.555 75.565) (width 1.4) (layer F.Cu) (net 0))
-  (segment (start 123.19 64.77) (end 123.19 74.93) (width 1.4) (layer F.Cu) (net 0))
+  (segment (start 123.19 76.2) (end 121.92 74.93) (width 1.4) (layer F.Cu) (net 0))
+  (segment (start 123.19 64.77) (end 123.19 76.2) (width 1.4) (layer F.Cu) (net 0))
   (segment (start 119.38 71.12) (end 119.38 66.04) (width 1.4) (layer F.Cu) (net 0))
   (segment (start 119.38 66.04) (end 120.65 67.31) (width 1.4) (layer F.Cu) (net 0))
@@
   (segment (start 62.23 27.94) (end 63.5 27.94) (width 1.4) (layer F.Cu) (net 0))
   (segment (start 64.77 30.42) (end 64.77 29.21) (width 1.4) (layer F.Cu) (net 0))
+  (segment (start 91.44 71.12) (end 95.25 71.12) (width 1.4) (layer F.Cu) (net 0))
+  (segment (start 95.25 71.12) (end 95.25 76.2) (width 1.4) (layer F.Cu) (net 0))
+  (segment (start 95.25 76.2) (end 106.68 76.2) (width 1.4) (layer F.Cu) (net 0))
+  (segment (start 88.9 73.66) (end 88.9 78.74) (width 1.4) (layer F.Cu) (net 0))
+  (segment (start 125.73 76.2) (end 114.3 76.2) (width 1.4) (layer F.Cu) (net 0))
+  (segment (start 114.3 76.2) (end 115.57 76.2) (width 1.4) (layer F.Cu) (net 0))
+  (segment (start 102.87 76.2) (end 114.3 76.2) (width 1.4) (layer F.Cu) (net 0))
+  (segment (start 121.92 74.93) (end 116.84 74.93) (width 1.4) (layer F.Cu) (net 0))
 )

Commit message: minor changes on hardware plate
Routing:
- net (no net): track 2095.2 -> 2096.7 mm
Changed lines of the file:
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@@
     (thickness 1.6)
     (drawings 7)
-    (tracks 464)
+    (tracks 467)
     (zones 0)
     (modules 63)
@@
   (segment (start 91.44 40.64) (end 91.44 39.37) (width 1.4) (layer F.Cu) (net 0))
   (segment (start 85.09 46.99) (end 91.44 40.64) (width 1.4) (layer F.Cu) (net 0))
-  (segment (start 91.44 36.83) (end 83.82 44.45) (width 1.4) (layer F.Cu) (net 0))
   (via (at 93.98 44.45) (size 2) (drill 1) (layers F.Cu B.Cu) (net 0))
   (segment (start 93.98 39.37) (end 93.98 44.45) (width 1.4) (layer F.Cu) (net 0))
@@
   (segment (start 102.87 76.2) (end 114.3 76.2) (width 1.4) (layer F.Cu) (net 0))
   (segment (start 121.92 74.93) (end 116.84 74.93) (width 1.4) (layer F.Cu) (net 0))
+  (segment (start 91.44 36.83) (end 88.9 36.83) (width 1.4) (layer F.Cu) (net 0))
+  (segment (start 88.9 36.83) (end 87.63 38.1) (width 1.4) (layer F.Cu) (net 0))
+  (segment (start 87.63 38.1) (end 87.63 40.64) (width 1.4) (layer F.Cu) (net 0))
+  (segment (start 87.63 40.64) (end 83.82 44.45) (width 1.4) (layer F.Cu) (net 0))
 )
